File: GettingToBlinky5.0.kicad_pcb (KiCad board)
At the start: 2 copper layers, 7 parts, among them U1 7555

Commit message: Completed Finishing The Layout Video
Parts:
- BT1: moved to B.Cu
- moved R3 37.2 mm to (139.0, 98.0), turned to 270 degrees
- moved C1 36.9 mm to (139.0, 93.5), turned to 90 degrees
- moved D1 29.2 mm to (139.0, 102.5), turned to 90 degrees
- moved U1 24.0 mm to (146.0, 97.0)
- moved R2 19.7 mm to (153.0, 100.5), turned to 270 degrees
- moved R1 14.3 mm to (153.0, 95.0), turned to 270 degrees
- moved BT1 1.75 mm to (146.1, 97.0)
Connections:
- net Net-(BT1-Pad1) renamed /VDD
- net Net-(C1-Pad1) renamed /THR
- net Net-(R1-Pad2) renamed /DIS
Routing:
- net /THR: track 0.00 -> 16.9 mm
- net /VDD: track 0.00 -> 12.8 mm, vias 0 -> 2
- net /DIS: track 0.00 -> 8.12 mm
- net Net-(R3-Pad1): track 0.00 -> 4.80 mm
- net GND: track 0.00 -> 4.36 mm, vias 0 -> 3
- net Net-(D1-Pad2): track 0.00 -> 2.45 mm
- added copper zone on F.Cu, net /VDD
- added copper zone on B.Cu, net GND
Other:
- board outline added: 32 x 30 mm

Commit message: Completed Output Files For Manufacturing Video
Other:
- board text added: "Getting To Blinky 5.0"
- board text added: "Made by Chris"
Changed lines of the file:
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@@
   (general
     (thickness 1.6)
-    (drawings 4)
+    (drawings 6)
     (tracks 32)
     (zones 0)
@@
     (46 B.CrtYd user)
     (47 F.CrtYd user)
-    (48 B.Fab user)
-    (49 F.Fab user)
+    (48 B.Fab user hide)
+    (49 F.Fab user hide)
   )
   (setup
@@
     (pcb_text_size 1.5 1.5)
     (mod_edge_width 0.12)
-    (mod_text_size 1 1)
+    (mod_text_size 1.3 1.3)
     (mod_text_width 0.15)
     (pad_size 1.524 1.524)
@@
       (psa4output false)
       (plotreference true)
-      (plotvalue true)
+      (plotvalue false)
       (plotinvisibletext false)
       (padsonsilk false)
@@
       (outputformat 1)
       (mirror false)
-      (drillshape 1)
+      (drillshape 0)
       (scaleselection 1)
-      (outputdirectory ""))
+      (outputdirectory "Gerbers/"))
   )
   (net 0 "")
@@
   (module GettingToBlinky5:S8211-46R (layer B.Cu)
     (at 146.05 97)
-    (fp_text reference BT1 (at 0 -4.05) (layer B.SilkS)
-      (effects (font (size 1 1) (thickness 0.15)) (justify mirror))
-    )
-    (fp_text value CR2032 (at 0.05 4) (layer B.Fab)
+    (fp_text reference BT1 (at -0.1 -9.05) (layer B.SilkS)
+      (effects (font (size 1.3 1.3) (thickness 0.15)) (justify mirror))
+    )
+    (fp_text value CR2032 (at 0.05 4) (layer B.Fab) hide
       (effects (font (size 1 1) (thickness 0.15)) (justify mirror))
     )
@@
     (attr smd)
     (fp_text reference U1 (at 0 -3.4) (layer F.SilkS)
-      (effects (font (size 1 1) (thickness 0.15)))
-    )
-    (fp_text value 7555 (at 0 3.4) (layer F.Fab)
+      (effects (font (size 1.3 1.3) (thickness 0.15)))
+    )
+    (fp_text value 7555 (at 0 3.4) (layer F.Fab) hide
       (effects (font (size 1 1) (thickness 0.15)))
     )
     (fp_text user %R (at 0 0) (layer F.Fab)
-      (effects (font (size 0.98 0.98) (thickness 0.15)))
+      (effects (font (size 1 1) (thickness 0.15)))
     )
     (fp_line (start 3.7 -2.7) (end -3.7 -2.7) (layer F.CrtYd) (width 0.05))
@@
     (tags "resistor handsolder")
     (attr smd)
-    (fp_text reference R3 (at 0 -1.65 90) (layer F.SilkS)
-      (effects (font (size 1 1) (thickness 0.15)))
-    )
-    (fp_text value 1K (at 0 1.65 90) (layer F.Fab)
-      (effects (font (size 1 1) (thickness 0.15)))
-    )
-    (fp_text user %R (at 0 0 90) (layer F.Fab)
-      (effects (font (size 0.5 0.5) (thickness 0.08)))
+    (fp_text reference R3 (at 0.05 1.95 90) (layer F.SilkS)
+      (effects (font (size 1.3 1.3) (thickness 0.15)))
+    )
+    (fp_text value 1K (at 0 1.65 90) (layer F.Fab) hide
+      (effects (font (size 1 1) (thickness 0.15)))
+    )
+    (fp_text user %R (at 0 0 90) (layer F.Fab)
+      (effects (font (size 1 1) (thickness 0.15)))
     )
     (fp_line (start 1.85 0.95) (end -1.85 0.95) (layer F.CrtYd) (width 0.05))
@@
     (tags "resistor handsolder")
     (attr smd)
-    (fp_text reference R2 (at 0 -1.65 90) (layer F.SilkS)
-      (effects (font (size 1 1) (thickness 0.15)))
-    )
-    (fp_text value 470K (at 0 1.65 90) (layer F.Fab)
-      (effects (font (size 1 1) (thickness 0.15)))
-    )
-    (fp_text user %R (at 0 0 90) (layer F.Fab)
-      (effects (font (size 0.5 0.5) (thickness 0.08)))
+    (fp_text reference R2 (at 0 -2.05 90) (layer F.SilkS)
+      (effects (font (size 1.3 1.3) (thickness 0.15)))
+    )
+    (fp_text value 470K (at 0 1.65 90) (layer F.Fab) hide
+      (effects (font (size 1 1) (thickness 0.15)))
+    )
+    (fp_text user %R (at 0 0 90) (layer F.Fab)
+      (effects (font (size 1 1) (thickness 0.15)))
     )
     (fp_line (start 1.85 0.95) (end -1.85 0.95) (layer F.CrtYd) (width 0.05))
@@
     (tags "resistor handsolder")
     (attr smd)
-    (fp_text reference R1 (at 0 -1.65 90) (layer F.SilkS)
-      (effects (font (size 1 1) (thickness 0.15)))
-    )
-    (fp_text value 1K (at 0 1.65 90) (layer F.Fab)
-      (effects (font (size 1 1) (thickness 0.15)))
-    )
-    (fp_text user %R (at 0 0 90) (layer F.Fab)
-      (effects (font (size 0.5 0.5) (thickness 0.08)))
+    (fp_text reference R1 (at 0 -2.05 90) (layer F.SilkS)
+      (effects (font (size 1.3 1.3) (thickness 0.15)))
+    )
+    (fp_text value 1K (at 0 1.65 90) (layer F.Fab) hide
+      (effects (font (size 1 1) (thickness 0.15)))
+    )
+    (fp_text user %R (at 0 0 90) (layer F.Fab)
+      (effects (font (size 1 1) (thickness 0.15)))
     )
     (fp_line (start 1.85 0.95) (end -1.85 0.95) (layer F.CrtYd) (width 0.05))
@@
     (tags "LED handsolder")
     (attr smd)
-    (fp_text reference D1 (at 0 -1.65 90) (layer F.SilkS)
-      (effects (font (size 1 1) (thickness 0.15)))
-    )
-    (fp_text value LED (at 0 1.65 90) (layer F.Fab)
-      (effects (font (size 1 1) (thickness 0.15)))
-    )
-    (fp_text user %R (at 0 0 90) (layer F.Fab)
-      (effects (font (size 0.5 0.5) (thickness 0.08)))
+    (fp_text reference D1 (at 0 -1.95 90) (layer F.SilkS)
+      (effects (font (size 1.3 1.3) (thickness 0.15)))
+    )
+    (fp_text value LED (at 0 1.65 90) (layer F.Fab) hide
+      (effects (font (size 1 1) (thickness 0.15)))
+    )
+    (fp_text user %R (at 0 0 90) (layer F.Fab)
+      (effects (font (size 1 1) (thickness 0.15)))
     )
     (fp_line (start 1.85 0.95) (end -1.85 0.95) (layer F.CrtYd) (width 0.05))
@@
     (tags "capacitor handsolder")
     (attr smd)
-    (fp_text reference C1 (at 0 -1.65 90) (layer F.SilkS)
-      (effects (font (size 1 1) (thickness 0.15)))
-    )
-    (fp_text value 1U (at 0 1.65 90) (layer F.Fab)
-      (effects (font (size 1 1) (thickness 0.15)))
-    )
-    (fp_text user %R (at 0 0 90) (layer F.Fab)
-      (effects (font (size 0.5 0.5) (thickness 0.08)))
+    (fp_text reference C1 (at 0 -1.95 90) (layer F.SilkS)
+      (effects (font (size 1.3 1.3) (thickness 0.15)))
+    )
+    (fp_text value 1U (at 0 1.65 90) (layer F.Fab) hide
+      (effects (font (size 1 1) (thickness 0.15)))
+    )
+    (fp_text user %R (at 0 0 90) (layer F.Fab)
+      (effects (font (size 1 1) (thickness 0.15)))
     )
     (fp_line (start 1.85 0.95) (end -1.85 0.95) (layer F.CrtYd) (width 0.05))
@@
     )
   )
+  (gr_text "Made by Chris" (at 146.25 108.45) (layer F.SilkS)
+    (effects (font (size 1.3 1.3) (thickness 0.15)))
+  )
+  (gr_text "Getting To Blinky 5.0" (at 146.25 85.8) (layer F.SilkS)
+    (effects (font (size 1.3 1.3) (thickness 0.15)))
+  )
   (gr_line (start 162 82) (end 130 82) (layer Edge.Cuts) (width 0.05))
